Commit message: Working simulation

File: ur_simulation_gazebo/urdf/ur_gazebo_classic.urdf.xacro (robot description, xacro)
@@ -14,11 +14,15 @@
    <xacro:arg name="visual_params" default="$(find ur_description)/config/$(arg ur_type)/visual_parameters.yaml"/>
    <xacro:arg name="joint_dynamics_params" default="$(find ur_description)/config/$(arg ur_type)/joint_dynamics_parameters.yaml"/>
+   <xacro:arg name="transmission_hw_interface" default=""/>
    <xacro:arg name="safety_limits" default="false"/>
    <xacro:arg name="safety_pos_margin" default="0.15"/>
    <xacro:arg name="safety_k_position" default="20"/>
    <xacro:arg name="simulation_controllers" default="" />
+   <!-- Initial positions for simulation -->
    <xacro:arg name="initial_positions_file" default="$(find ur_simulation_gazebo)/config/home_positions.yaml"/>
    <!-- convert to property to use substitution in function -->
    <xacro:property name="initial_positions_file" default="$(arg initial_positions_file)"/>
+   <!-- create link fixed to the "world" -->
+   <link name="world"/>
    <xacro:read_model_data
      joint_limits_parameters_file="$(arg joint_limit_params)"
@@ -34,4 +38,5 @@
       the effort limits are loaded by read_model_data
    -->
+   <!-- arm instance -->
    <xacro:ur_robot
      name="$(arg name)"
@@ -44,4 +49,5 @@
      <origin xyz="0 0 0.05" rpy="0 0 0" />          <!-- position robot in the world, a little elevated to avoid base contact-->
    </xacro:ur_robot>
+   <!-- ros2 control, if needed -->
    <xacro:ur_ros2_control
       name="$(arg name)" prefix="$(arg prefix)"
@@ -57,3 +63,11 @@
       </ros2_control_hardware>
    </xacro:ur_ros2_control>
+   <!-- now gazebo tags can just be in the gazebo package. No switching needed in ur_description -->
+   <gazebo reference="world">
+   </gazebo>
+   <gazebo>
+      <plugin filename="libgazebo_ros2_control.so" name="gazebo_ros2_control">
+         <parameters>$(arg simulation_controllers)</parameters>
+      </plugin>
+   </gazebo>
 </robot>

Commit message: Working friction stabilization

File: ur_simulation_gazebo/urdf/ur_gazebo_classic.urdf.xacro (robot description, xacro)
@@ -33,9 +33,18 @@
      force_abs_paths="false"/>
    <!--
+      See https://github.com/UniversalRobots/Universal_Robots_ROS2_Gazebo_Simulation/issues/19
+      We need to set fmax for ODE.
       Joint dynamics damping and friction default to zero (from ur_description/config files)
       To address #19, we could define the joint dynamics in a config file,
       but it does seem good to use some multiple of the effort limit
-      the effort limits are loaded by read_model_data
+      the effort limits are loaded by read_model_data and reside at this file's scope
+      so we can compute them on the fly here
    -->
+   <xacro:property name="shoulder_pan_friction" value="${shoulder_pan_effort_limit*100.0}"/>
+   <xacro:property name="shoulder_lift_friction" value="${shoulder_lift_effort_limit*100.0}"/>
+   <xacro:property name="elbow_joint_friction" value="${elbow_joint_effort_limit*100.0}"/>
+   <xacro:property name="wrist_1_friction" value="${wrist_1_effort_limit*100.0}"/>
+   <xacro:property name="wrist_2_friction" value="${wrist_2_effort_limit*100.0}"/>
+   <xacro:property name="wrist_3_friction" value="${wrist_3_effort_limit*100.0}"/>
    <!-- arm instance -->
    <xacro:ur_robot
